File: circuito/CiruitoKicad/iceCubeNomeFeio.sch (KiCad schematic (older format))
At the start: 25 parts, among them J1 VIN, J10 MB, J2 BLE, J3 2Y0A21, J4 2Y0A21, J5 2Y0A21, J6 2Y0A21, J7 aersrd, J8 adsfgd, J9 MA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

Commit message: finalizar circuito
Connections:
- net A15: now also U2.24 (PB15), U3.14 (INA1); no longer U2.30 (PA15), U3.11 (INB2)
- net B12: now reaches U2.21 (PB12)
- net B12: now also U3.11 (INB2)
- net B13: now reaches U2.22 (PB13)
- net B13: now also U3.12 (INB1)
- net B14: now reaches U2.23 (PB14)
- net B14: now also U3.13 (STNDBY)
- net A8: now reaches U2.25 (PA8)
- net A8: now also U3.15 (INA2)
- net B3: no longer names the net of U2.31 (PB3)
- net B3: no longer U3.12 (INB1)
- net B4: no longer names the net of U2.32 (PB4)
- net B4: no longer U3.13 (STNDBY)
- net B6: no longer names the net of U2.34 (PB6)
- net B6: no longer U3.14 (INA1)
- net B7: no longer names the net of U2.35 (PB7)
- net B7: no longer U3.15 (INA2)
- no-connect marks 19 -> 16
Changed lines of the file:
@@
 $EndDescr
-$Comp
-L MyLib-ALL:STM32F103C8T6 U2
-U 1 1 5D4212E5
-P 1850 4250
-F 0 "U2" H 2350 4365 50  0000 C CNN
-F 1 "STM32F103C8T6" H 2350 4274 50  0000 C CNN
-F 2 "MyFootprint:stm32f103c8t6-module-china" H 1850 4250 50  0001 C CNN
-F 3 "" H 1850 4250 50  0001 C CNN
-	1    1850 4250
-	1    0    0    -1
-$EndComp
 $Comp
 L MyLib-ALL:DC-DC U1
@@
 $EndComp
 Wire Wire Line
-	3050 6450 3050 4550
-Wire Wire Line
 	3050 4550 3000 4550
 NoConn ~ 3000 5150
 NoConn ~ 3000 5550
 NoConn ~ 3000 5650
-NoConn ~ 3000 6150
-NoConn ~ 3000 6250
-NoConn ~ 3000 6350
 $Comp
 L Connector:Conn_01x04_Female J2
@@
 	1    0    0    -1
 $EndComp
-Text HLabel 3100 4950 2    50   Output ~ 0
-B7
-Text HLabel 3100 5050 2    50   Output ~ 0
-B6
-Text HLabel 3100 5250 2    50   Output ~ 0
-B4
-Text HLabel 3100 5350 2    50   Output ~ 0
-B3
-Text HLabel 3100 5450 2    50   Output ~ 0
+Text HLabel 3150 6250 2    50   Output ~ 0
+B13
+Text HLabel 3150 6350 2    50   Output ~ 0
+B12
+Text HLabel 3150 5950 2    50   Output ~ 0
+A8
+Text HLabel 3150 6050 2    50   Output ~ 0
 A15
-Wire Wire Line
-	3100 5250 3000 5250
-Wire Wire Line
-	3000 5350 3100 5350
-Wire Wire Line
-	3100 5450 3000 5450
-Wire Wire Line
-	3000 5050 3100 5050
-Wire Wire Line
-	3100 4950 3000 4950
+Text HLabel 3150 6150 2    50   Output ~ 0
+B14
+Wire Wire Line
+	3150 5950 3000 5950
+Wire Wire Line
+	3000 6050 3150 6050
+Wire Wire Line
+	3150 6150 3000 6150
+Wire Wire Line
+	3000 6350 3150 6350
+Wire Wire Line
+	3150 6250 3000 6250
 $Comp
 L Connector:Conn_01x02_Female J9
@@
 Wire Wire Line
 	9700 2750 9700 2600
-Text HLabel 9400 2750 3    50   Input ~ 0
-B4
-Text HLabel 9300 2750 3    50   Input ~ 0
-B3
-Text HLabel 9200 2750 3    50   Input ~ 0
-A15
-Wire Wire Line
-	9400 2750 9400 2600
-Wire Wire Line
-	9300 2600 9300 2750
-Wire Wire Line
-	9200 2750 9200 2600
-Text HLabel 9600 2750 3    50   Input ~ 0
-B7
-Text HLabel 9500 2750 3    50   Input ~ 0
-B6
-Wire Wire Line
-	9600 2750 9600 2600
-Wire Wire Line
-	9500 2600 9500 2750
 NoConn ~ 3000 4850
 NoConn ~ 3000 4750
@@
 	0    -1   -1   0
 $EndComp
+Wire Wire Line
+	3050 6450 3050 4550
+$Comp
+L MyLib-ALL:STM32F103C8T6 U2
+U 1 1 5D4212E5
+P 1850 4250
+F 0 "U2" H 2350 4365 50  0000 C CNN
+F 1 "STM32F103C8T6" H 2350 4274 50  0000 C CNN
+F 2 "MyFootprint:stm32f103c8t6-module-china" H 1850 4250 50  0001 C CNN
+F 3 "" H 1850 4250 50  0001 C CNN
+	1    1850 4250
+	1    0    0    -1
+$EndComp
+Text HLabel 9300 2750 3    50   Input ~ 0
+B13
+Text HLabel 9200 2750 3    50   Input ~ 0
+B12
+Text HLabel 9600 2750 3    50   Input ~ 0
+A8
+Text HLabel 9500 2750 3    50   Input ~ 0
+A15
+Text HLabel 9400 2750 3    50   Input ~ 0
+B14
+Wire Wire Line
+	9600 2750 9600 2600
+Wire Wire Line
+	9200 2750 9200 2600
+Wire Wire Line
+	9300 2600 9300 2750
+Wire Wire Line
+	9400 2750 9400 2600
+Wire Wire Line
+	9500 2600 9500 2750
 $EndSCHEMATC

Commit message: organizando
Parts:
- U1: symbol MyLib-ALL:DC-DC -> iceCubeNomeFeio-rescue:DC-DC-MyLib-ALL
- U2: symbol MyLib-ALL:STM32F103C8T6 -> iceCubeNomeFeio-rescue:STM32F103C8T6-MyLib-ALL
- U3: symbol MyLib-ALL:TB6612FNG -> iceCubeNomeFeio-rescue:TB6612FNG-MyLib-ALL
Connections:
- net +5V: now also U1.1 (VOUT); no longer U1.4 (VOUT)
- net VIM: now also U1.4 (VIN); no longer U1.1 (VIN)
- net A15 renamed B15
Changed lines of the file:
@@
 $EndDescr
 $Comp
-L MyLib-ALL:DC-DC U1
+L iceCubeNomeFeio-rescue:DC-DC-MyLib-ALL U1
 U 1 1 5D42142E
 P 1300 2850
@@
 $EndComp
 $Comp
-L 4V2:+5V #PWR07
+L iceCubeNomeFeio-rescue:+5V-4V2 #PWR07
 U 1 1 5D422A39
 P 4150 1300
@@
 $EndComp
 $Comp
-L 4V2:Earth #PWR09
+L iceCubeNomeFeio-rescue:Earth-4V2 #PWR09
 U 1 1 5D422B44
 P 4250 1300
@@
 $EndComp
 $Comp
-L 4V2:+5V #PWR010
+L iceCubeNomeFeio-rescue:+5V-4V2 #PWR010
 U 1 1 5D422E52
 P 4600 1300
@@
 $EndComp
 $Comp
-L 4V2:Earth #PWR011
+L iceCubeNomeFeio-rescue:Earth-4V2 #PWR011
 U 1 1 5D422E58
 P 4700 1300
@@
 $EndComp
 $Comp
-L 4V2:+5V #PWR013
+L iceCubeNomeFeio-rescue:+5V-4V2 #PWR013
 U 1 1 5D422FEF
 P 5050 1300
@@
 $EndComp
 $Comp
-L 4V2:Earth #PWR014
+L iceCubeNomeFeio-rescue:Earth-4V2 #PWR014
 U 1 1 5D422FF5
 P 5150 1300
@@
 $EndComp
 $Comp
-L 4V2:+5V #PWR015
+L iceCubeNomeFeio-rescue:+5V-4V2 #PWR015
 U 1 1 5D423006
 P 5500 1300
@@
 $EndComp
 $Comp
-L 4V2:Earth #PWR017
+L iceCubeNomeFeio-rescue:Earth-4V2 #PWR017
 U 1 1 5D42300C
 P 5600 1300
@@
 	5700 1300 5700 1150
 $Comp
-L 4V2:+5V #PWR020
+L iceCubeNomeFeio-rescue:+5V-4V2 #PWR020
 U 1 1 5D424281
 P 6250 1300
@@
 $EndComp
 $Comp
-L 4V2:Earth #PWR018
+L iceCubeNomeFeio-rescue:Earth-4V2 #PWR018
 U 1 1 5D424287
 P 6150 1300
@@
 	6050 1300 6050 1150
 $Comp
-L 4V2:+5V #PWR022
+L iceCubeNomeFeio-rescue:+5V-4V2 #PWR022
 U 1 1 5D424F2E
 P 6800 1300
@@
 $EndComp
 $Comp
-L 4V2:Earth #PWR021
+L iceCubeNomeFeio-rescue:Earth-4V2 #PWR021
 U 1 1 5D424F34
 P 6700 1300
@@
 $EndComp
 $Comp
-L 4V2:Earth #PWR08
+L iceCubeNomeFeio-rescue:Earth-4V2 #PWR08
 U 1 1 5D4256F1
 P 4200 3000
@@
 $EndComp
 $Comp
-L 4V2:Earth #PWR012
+L iceCubeNomeFeio-rescue:Earth-4V2 #PWR012
 U 1 1 5D42963D
 P 4650 3000
@@
 $EndComp
 $Comp
-L 4V2:Earth #PWR016
+L iceCubeNomeFeio-rescue:Earth-4V2 #PWR016
 U 1 1 5D42A644
 P 5100 3000
@@
 $EndComp
 $Comp
-L 4V2:Earth #PWR019
+L iceCubeNomeFeio-rescue:Earth-4V2 #PWR019
 U 1 1 5D42A661
 P 5550 3000
@@
 $EndComp
 $Comp
-L 4V2:Earth #PWR023
+L iceCubeNomeFeio-rescue:Earth-4V2 #PWR023
 U 1 1 5D42B44C
 P 6000 3000
@@
 $EndComp
 $Comp
-L 4V2:Earth #PWR024
+L iceCubeNomeFeio-rescue:Earth-4V2 #PWR024
 U 1 1 5D42B469
 P 6450 3000
@@
 OUT6
 $Comp
-L 4V2:Earth #PWR02
+L iceCubeNomeFeio-rescue:Earth-4V2 #PWR02
 U 1 1 5D434B34
 P 1000 2850
@@
 	1000 2800 1100 2800
 $Comp
-L 4V2:Earth #PWR04
+L iceCubeNomeFeio-rescue:Earth-4V2 #PWR04
 U 1 1 5D435CCF
 P 2200 2850
@@
 	2200 2700 2100 2700
 $Comp
-L 4V2:+5V #PWR03
+L iceCubeNomeFeio-rescue:+5V-4V2 #PWR03
 U 1 1 5D437462
 P 2200 2100
@@
 $EndComp
 $Comp
-L 4V2:Earth #PWR01
+L iceCubeNomeFeio-rescue:Earth-4V2 #PWR01
 U 1 1 5D43E251
 P 950 1800
@@
 	1000 2500 1100 2500
 $Comp
-L 4V2:+5V #PWR029
+L iceCubeNomeFeio-rescue:+5V-4V2 #PWR029
 U 1 1 5D449A75
 P 3150 4150
@@
 NoConn ~ 1700 6050
 $Comp
-L 4V2:Earth #PWR025
+L iceCubeNomeFeio-rescue:Earth-4V2 #PWR025
 U 1 1 5D4738B2
 P 1600 6450
@@
 	1600 6350 1600 6250
 $Comp
-L 4V2:Earth #PWR028
+L iceCubeNomeFeio-rescue:Earth-4V2 #PWR028
 U 1 1 5D476C14
 P 3050 6450
@@
 $EndComp
 $Comp
-L 4V2:+5V #PWR06
+L iceCubeNomeFeio-rescue:+5V-4V2 #PWR06
 U 1 1 5D491E8B
 P 3400 1400
@@
 $EndComp
 $Comp
-L 4V2:Earth #PWR05
+L iceCubeNomeFeio-rescue:Earth-4V2 #PWR05
 U 1 1 5D491F65
 P 3300 1400
@@
 	3150 5850 3000 5850
 $Comp
-L 4V2:Earth #PWR030
+L iceCubeNomeFeio-rescue:Earth-4V2 #PWR030
 U 1 1 5D4BA922
 P 8800 2900
@@
 $EndComp
 $Comp
-L MyLib-ALL:TB6612FNG U3
+L iceCubeNomeFeio-rescue:TB6612FNG-MyLib-ALL U3
 U 1 1 5D4DB153
 P 9800 1550
@@
 	9600 1400 9600 1450
 $Comp
-L 4V2:+5V #PWR027
+L iceCubeNomeFeio-rescue:+5V-4V2 #PWR027
 U 1 1 5D4F17D7
 P 9650 1100
@@
 A8
 Text HLabel 3150 6050 2    50   Output ~ 0
-A15
+B15
 Text HLabel 3150 6150 2    50   Output ~ 0
 B14
@@
 	3050 6450 3050 4550
 $Comp
-L MyLib-ALL:STM32F103C8T6 U2
+L iceCubeNomeFeio-rescue:STM32F103C8T6-MyLib-ALL U2
 U 1 1 5D4212E5
 P 1850 4250
@@
 A8
 Text HLabel 9500 2750 3    50   Input ~ 0
-A15
+B15
 Text HLabel 9400 2750 3    50   Input ~ 0
 B14
