File: circuito/CiruitoKicad/iceCubeNomeFeio.kicad_pcb (KiCad board)
At the start: 2 copper layers, 56 x 57 mm, 25 parts, among them J1 VIN, J10 MB, J2 BLE, J3 2Y0A21, J4 2Y0A21, J5 2Y0A21, J6 2Y0A21, J7 2Y0A21, J8 2Y0A21, J9 MA, U1 DC-DC, U2 STM32F103C8T6, U3 TB6612FNG

Commit message: finalizar circuito
Parts:
- J7: value 2Y0A21 -> aersrd
- J8: value 2Y0A21 -> adsfgd
- moved R2 42.6 mm to (132.0, 68.0), turned to 180 degrees
- moved R3 34.3 mm to (132.0, 74.5)
- moved R9 33.8 mm to (130.5, 117.5)
- moved R12 32.6 mm to (130.5, 105.5), turned to 180 degrees
- moved R11 28.8 mm to (130.5, 108.5)
- moved R10 21.9 mm to (130.5, 115.0), turned to 180 degrees
- moved R4 18.7 mm to (132.0, 78.5), turned to 180 degrees
- moved R5 17.1 mm to (130.5, 84.0)
- moved J1 14.0 mm to (172.0, 93.0)
- moved J10 14.0 mm to (158.0, 93.0)
- moved R8 13.1 mm to (132.0, 96.5), turned to 180 degrees
- moved R1 12.7 mm to (132.0, 65.0)
- moved R6 9.71 mm to (130.5, 87.0), turned to 180 degrees
- moved J8 9.54 mm to (125.0, 108.0)
- moved J7 9.46 mm to (125.0, 117.5)
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Connections:
- U2 pad 21: Net-(U2-Pad21) -> /B12
- U2 pad 22: Net-(U2-Pad22) -> /B13
- U2 pad 23: Net-(U2-Pad23) -> /B14
- U2 pad 24: Net-(U2-Pad24) -> /A15
- U2 pad 25: Net-(U2-Pad25) -> /A8
- U2 pad 30: /A15 -> Net-(U2-Pad30)
- U2 pad 31: /B3 -> Net-(U2-Pad31)
- U2 pad 32: /B4 -> Net-(U2-Pad32)
- U2 pad 34: /B6 -> Net-(U2-Pad34)
- U2 pad 35: /B7 -> Net-(U2-Pad35)
- U3 pad 11: /A15 -> /B12
- U3 pad 12: /B3 -> /B13
- U3 pad 13: /B4 -> /B14
- U3 pad 14: /B6 -> /A15
- U3 pad 15: /B7 -> /A8
Routing:
- net +5V: track 0.00 -> 201.9 mm
- net /RXD: track 0.00 -> 39.3 mm
- net /TXD: track 0.00 -> 38.9 mm
- net /OUT5M: track 0.00 -> 34.5 mm
- net /A10: track 0.00 -> 34.5 mm
- net /A9: track 0.00 -> 31.0 mm
- net /A8: track 0.00 -> 29.5 mm
- net /A15: track 0.00 -> 26.8 mm
- net /B14: track 0.00 -> 23.3 mm
- net /OUT6M: track 0.00 -> 21.6 mm
- net /B13: track 0.00 -> 20.2 mm
- net /VIM: track 0.00 -> 18.0 mm
- net /B12: track 0.00 -> 16.9 mm
- net /OUT4M: track 0.00 -> 14.7 mm
- net /OUT1M: track 0.00 -> 12.2 mm
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- added copper zone on B.Cu, net Earth

Commit message: organizando
Parts:
- moved R3 3.54 mm to (131.5, 71.0)
- moved R4 3.54 mm to (131.5, 75.0)
- moved J1 3.54 mm to (172.5, 89.5)
- moved J10 3.54 mm to (158.5, 89.5)
- moved J2 3.54 mm to (157.5, 69.5)
- moved J3 3.54 mm to (125.5, 66.6)
- moved J4 3.54 mm to (125.5, 76.1)
- moved J5 3.54 mm to (125.5, 85.6)
- moved J6 3.54 mm to (125.5, 95.1)
- moved J7 3.54 mm to (125.5, 114.0)
- moved J8 3.54 mm to (125.5, 104.5)
- moved J9 3.54 mm to (165.5, 89.5)
- moved R1 3.54 mm to (132.5, 61.5)
- moved R10 3.54 mm to (131.0, 111.5)
- moved R11 3.54 mm to (131.0, 105.0)
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Connections:
- U1 pad 1: /VIM -> +5V
- U1 pad 4: +5V -> /VIM
Routing:
- net /TXD: track 38.9 -> 57.6 mm
- net /VIM: track 18.0 -> 31.8 mm
- net Earth: track 10.1 -> 0.75 mm, vias 1 -> 0
- net /RXD: track 39.3 -> 45.5 mm
- net /A9: track 31.0 -> 36.3 mm
- net /OUT2M: track 9.03 -> 12.2 mm
- net /A10: track 34.5 -> 31.8 mm
- net /B13: track 20.2 -> 22.8 mm
- net /A8: track 29.5 -> 27.2 mm
- net /B14: track 23.3 -> 25.4 mm
- net /A15: track 26.8 -> 24.7 mm
- net /OUT5M: track 34.5 -> 35.8 mm
- net +5V: track 201.9 -> 200.8 mm
- net /OUT4M: track 14.7 -> 15.7 mm
- net /OUT2: track 6.00 -> 4.97 mm
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Other:
- board text added: "5"
- board text added: "@pedro_ibs Robo IceCube"
- board text added: "USB"
- board text added: "VIN"

Commit message: att PCB
Parts:
- added J1: VIN, Connector_Molex:Molex_KK-254_AE-6410-02A_1x02_P2.54mm_Vertical, F.Cu at (72.5, 119.5)
- added J1: VIN, Connector_Molex:Molex_KK-254_AE-6410-02A_1x02_P2.54mm_Vertical, F.Cu at (212.5, 119.5)
- added J1: VIN, Connector_Molex:Molex_KK-254_AE-6410-02A_1x02_P2.54mm_Vertical, F.Cu at (142.5, 119.5)
- added J1: VIN, Connector_Molex:Molex_KK-254_AE-6410-02A_1x02_P2.54mm_Vertical, F.Cu at (212.5, 49.5)
- added J1: VIN, Connector_Molex:Molex_KK-254_AE-6410-02A_1x02_P2.54mm_Vertical, F.Cu at (142.5, 49.5)
- added J10: MB, Connector_Molex:Molex_KK-254_AE-6410-02A_1x02_P2.54mm_Vertical, F.Cu at (128.5, 119.5)
- added J10: MB, Connector_Molex:Molex_KK-254_AE-6410-02A_1x02_P2.54mm_Vertical, F.Cu at (198.5, 119.5)
- added J10: MB, Connector_Molex:Molex_KK-254_AE-6410-02A_1x02_P2.54mm_Vertical, F.Cu at (58.5, 119.5)
- added J10: MB, Connector_Molex:Molex_KK-254_AE-6410-02A_1x02_P2.54mm_Vertical, F.Cu at (198.5, 49.5)
- added J10: MB, Connector_Molex:Molex_KK-254_AE-6410-02A_1x02_P2.54mm_Vertical, F.Cu at (128.5, 49.5)
- added J2: BLE, Connector_PinSocket_2.54mm:PinSocket_1x04_P2.54mm_Vertical, F.Cu at (57.5, 99.5)
- added J2: BLE, Connector_PinSocket_2.54mm:PinSocket_1x04_P2.54mm_Vertical, F.Cu at (127.5, 99.5)
- added J2: BLE, Connector_PinSocket_2.54mm:PinSocket_1x04_P2.54mm_Vertical, F.Cu at (197.5, 99.5)
- added J2: BLE, Connector_PinSocket_2.54mm:PinSocket_1x04_P2.54mm_Vertical, F.Cu at (197.5, 29.5)
- added J2: BLE, Connector_PinSocket_2.54mm:PinSocket_1x04_P2.54mm_Vertical, F.Cu at (127.5, 29.5)
- added J3: 2Y0A21, Connector_Molex:Molex_KK-254_AE-6410-03A_1x03_P2.54mm_Vertical, F.Cu at (25.5, 96.6)
- added J3: 2Y0A21, Connector_Molex:Molex_KK-254_AE-6410-03A_1x03_P2.54mm_Vertical, F.Cu at (95.5, 96.6)
- added J3: 2Y0A21, Connector_Molex:Molex_KK-254_AE-6410-03A_1x03_P2.54mm_Vertical, F.Cu at (165.5, 96.6)
- added J3: 2Y0A21, Connector_Molex:Molex_KK-254_AE-6410-03A_1x03_P2.54mm_Vertical, F.Cu at (165.5, 26.6)
- added J3: 2Y0A21, Connector_Molex:Molex_KK-254_AE-6410-03A_1x03_P2.54mm_Vertical, F.Cu at (95.5, 26.6)
- added J4: 2Y0A21, Connector_Molex:Molex_KK-254_AE-6410-03A_1x03_P2.54mm_Vertical, F.Cu at (25.5, 106.1)
- added J4: 2Y0A21, Connector_Molex:Molex_KK-254_AE-6410-03A_1x03_P2.54mm_Vertical, F.Cu at (95.5, 106.1)
- added J4: 2Y0A21, Connector_Molex:Molex_KK-254_AE-6410-03A_1x03_P2.54mm_Vertical, F.Cu at (165.5, 106.1)
- added J4: 2Y0A21, Connector_Molex:Molex_KK-254_AE-6410-03A_1x03_P2.54mm_Vertical, F.Cu at (165.5, 36.1)
- added J4: 2Y0A21, Connector_Molex:Molex_KK-254_AE-6410-03A_1x03_P2.54mm_Vertical, F.Cu at (95.5, 36.1)
- added J5: 2Y0A21, Connector_Molex:Molex_KK-254_AE-6410-03A_1x03_P2.54mm_Vertical, F.Cu at (25.5, 115.6)
- added J5: 2Y0A21, Connector_Molex:Molex_KK-254_AE-6410-03A_1x03_P2.54mm_Vertical, F.Cu at (165.5, 115.6)
- added J5: 2Y0A21, Connector_Molex:Molex_KK-254_AE-6410-03A_1x03_P2.54mm_Vertical, F.Cu at (95.5, 115.6)
- added J5: 2Y0A21, Connector_Molex:Molex_KK-254_AE-6410-03A_1x03_P2.54mm_Vertical, F.Cu at (165.5, 45.6)
- added J5: 2Y0A21, Connector_Molex:Molex_KK-254_AE-6410-03A_1x03_P2.54mm_Vertical, F.Cu at (95.5, 45.6)
- added J6: 2Y0A21, Connector_Molex:Molex_KK-254_AE-6410-03A_1x03_P2.54mm_Vertical, F.Cu at (165.5, 125.1)
- added J6: 2Y0A21, Connector_Molex:Molex_KK-254_AE-6410-03A_1x03_P2.54mm_Vertical, F.Cu at (95.5, 125.1)
- added J6: 2Y0A21, Connector_Molex:Molex_KK-254_AE-6410-03A_1x03_P2.54mm_Vertical, F.Cu at (25.5, 125.1)
- added J6: 2Y0A21, Connector_Molex:Molex_KK-254_AE-6410-03A_1x03_P2.54mm_Vertical, F.Cu at (165.5, 55.1)
- added J6: 2Y0A21, Connector_Molex:Molex_KK-254_AE-6410-03A_1x03_P2.54mm_Vertical, F.Cu at (95.5, 55.1)
- added J7: aersrd, Connector_Molex:Molex_KK-254_AE-6410-03A_1x03_P2.54mm_Vertical, F.Cu at (25.5, 144.0)
- added J7: aersrd, Connector_Molex:Molex_KK-254_AE-6410-03A_1x03_P2.54mm_Vertical, F.Cu at (165.5, 144.0)
- added J7: aersrd, Connector_Molex:Molex_KK-254_AE-6410-03A_1x03_P2.54mm_Vertical, F.Cu at (95.5, 144.0)
- added J7: aersrd, Connector_Molex:Molex_KK-254_AE-6410-03A_1x03_P2.54mm_Vertical, F.Cu at (165.5, 74.0)
- added J7: aersrd, Connector_Molex:Molex_KK-254_AE-6410-03A_1x03_P2.54mm_Vertical, F.Cu at (95.5, 74.0)
- added J8: adsfgd, Connector_Molex:Molex_KK-254_AE-6410-03A_1x03_P2.54mm_Vertical, F.Cu at (95.5, 134.5)
- added J8: adsfgd, Connector_Molex:Molex_KK-254_AE-6410-03A_1x03_P2.54mm_Vertical, F.Cu at (25.5, 134.5)
- added J8: adsfgd, Connector_Molex:Molex_KK-254_AE-6410-03A_1x03_P2.54mm_Vertical, F.Cu at (165.5, 134.5)
- added J8: adsfgd, Connector_Molex:Molex_KK-254_AE-6410-03A_1x03_P2.54mm_Vertical, F.Cu at (165.5, 64.5)
- added J8: adsfgd, Connector_Molex:Molex_KK-254_AE-6410-03A_1x03_P2.54mm_Vertical, F.Cu at (95.5, 64.5)
- added J9: MA, Connector_Molex:Molex_KK-254_AE-6410-02A_1x02_P2.54mm_Vertical, F.Cu at (65.5, 119.5)
- added J9: MA, Connector_Molex:Molex_KK-254_AE-6410-02A_1x02_P2.54mm_Vertical, F.Cu at (205.5, 119.5)
- added J9: MA, Connector_Molex:Molex_KK-254_AE-6410-02A_1x02_P2.54mm_Vertical, F.Cu at (135.5, 119.5)
- added J9: MA, Connector_Molex:Molex_KK-254_AE-6410-02A_1x02_P2.54mm_Vertical, F.Cu at (205.5, 49.5)
- added J9: MA, Connector_Molex:Molex_KK-254_AE-6410-02A_1x02_P2.54mm_Vertical, F.Cu at (135.5, 49.5)
- added R1: 1K, Resistor_SMD:R_0805_2012Metric_Pad1.15x1.40mm_HandSolder, B.Cu at (32.5, 91.5)
- added R1: 1K, Resistor_SMD:R_0805_2012Metric_Pad1.15x1.40mm_HandSolder, B.Cu at (102.5, 91.5)
- added R1: 1K, Resistor_SMD:R_0805_2012Metric_Pad1.15x1.40mm_HandSolder, B.Cu at (172.5, 91.5)
- added R1: 1K, Resistor_SMD:R_0805_2012Metric_Pad1.15x1.40mm_HandSolder, B.Cu at (172.5, 21.5)
- added R1: 1K, Resistor_SMD:R_0805_2012Metric_Pad1.15x1.40mm_HandSolder, B.Cu at (102.5, 21.5)
- added R10: 2K, Resistor_SMD:R_0805_2012Metric_Pad1.15x1.40mm_HandSolder, B.Cu at (31.0, 141.5)
- added R10: 2K, Resistor_SMD:R_0805_2012Metric_Pad1.15x1.40mm_HandSolder, B.Cu at (171.0, 141.5)
- added R10: 2K, Resistor_SMD:R_0805_2012Metric_Pad1.15x1.40mm_HandSolder, B.Cu at (101.0, 141.5)
- added R10: 2K, Resistor_SMD:R_0805_2012Metric_Pad1.15x1.40mm_HandSolder, B.Cu at (171.0, 71.5)
- added R10: 2K, Resistor_SMD:R_0805_2012Metric_Pad1.15x1.40mm_HandSolder, B.Cu at (101.0, 71.5)
- added R11: 1K, Resistor_SMD:R_0805_2012Metric_Pad1.15x1.40mm_HandSolder, B.Cu at (171.0, 135.0)
- added R11: 1K, Resistor_SMD:R_0805_2012Metric_Pad1.15x1.40mm_HandSolder, B.Cu at (101.0, 135.0)
- added R11: 1K, Resistor_SMD:R_0805_2012Metric_Pad1.15x1.40mm_HandSolder, B.Cu at (31.0, 135.0)
- added R11: 1K, Resistor_SMD:R_0805_2012Metric_Pad1.15x1.40mm_HandSolder, B.Cu at (171.0, 65.0)
- added R11: 1K, Resistor_SMD:R_0805_2012Metric_Pad1.15x1.40mm_HandSolder, B.Cu at (101.0, 65.0)
- added R12: 2K, Resistor_SMD:R_0805_2012Metric_Pad1.15x1.40mm_HandSolder, B.Cu at (171.0, 132.0)
- added R12: 2K, Resistor_SMD:R_0805_2012Metric_Pad1.15x1.40mm_HandSolder, B.Cu at (31.0, 132.0)
- added R12: 2K, Resistor_SMD:R_0805_2012Metric_Pad1.15x1.40mm_HandSolder, B.Cu at (101.0, 132.0)
- added R12: 2K, Resistor_SMD:R_0805_2012Metric_Pad1.15x1.40mm_HandSolder, B.Cu at (171.0, 62.0)
- added R12: 2K, Resistor_SMD:R_0805_2012Metric_Pad1.15x1.40mm_HandSolder, B.Cu at (101.0, 62.0)
- added R2: 2K, Resistor_SMD:R_0805_2012Metric_Pad1.15x1.40mm_HandSolder, B.Cu at (172.5, 94.5)
- added R2: 2K, Resistor_SMD:R_0805_2012Metric_Pad1.15x1.40mm_HandSolder, B.Cu at (102.5, 94.5)
- added R2: 2K, Resistor_SMD:R_0805_2012Metric_Pad1.15x1.40mm_HandSolder, B.Cu at (32.5, 94.5)
- added R2: 2K, Resistor_SMD:R_0805_2012Metric_Pad1.15x1.40mm_HandSolder, B.Cu at (172.5, 24.5)
- added R2: 2K, Resistor_SMD:R_0805_2012Metric_Pad1.15x1.40mm_HandSolder, B.Cu at (102.5, 24.5)
- added R3: 1K, Resistor_SMD:R_0805_2012Metric_Pad1.15x1.40mm_HandSolder, B.Cu at (31.5, 101.0)
- added R3: 1K, Resistor_SMD:R_0805_2012Metric_Pad1.15x1.40mm_HandSolder, B.Cu at (171.5, 101.0)
- added R3: 1K, Resistor_SMD:R_0805_2012Metric_Pad1.15x1.40mm_HandSolder, B.Cu at (101.5, 101.0)
- added R3: 1K, Resistor_SMD:R_0805_2012Metric_Pad1.15x1.40mm_HandSolder, B.Cu at (171.5, 31.0)
- added R3: 1K, Resistor_SMD:R_0805_2012Metric_Pad1.15x1.40mm_HandSolder, B.Cu at (101.5, 31.0)
- added R4: 2K, Resistor_SMD:R_0805_2012Metric_Pad1.15x1.40mm_HandSolder, B.Cu at (171.5, 105.0)
- added R4: 2K, Resistor_SMD:R_0805_2012Metric_Pad1.15x1.40mm_HandSolder, B.Cu at (101.5, 105.0)
- added R4: 2K, Resistor_SMD:R_0805_2012Metric_Pad1.15x1.40mm_HandSolder, B.Cu at (31.5, 105.0)
- added R4: 2K, Resistor_SMD:R_0805_2012Metric_Pad1.15x1.40mm_HandSolder, B.Cu at (171.5, 35.0)
- added R4: 2K, Resistor_SMD:R_0805_2012Metric_Pad1.15x1.40mm_HandSolder, B.Cu at (101.5, 35.0)
- added R5: 1K, Resistor_SMD:R_0805_2012Metric_Pad1.15x1.40mm_HandSolder, B.Cu at (171.0, 110.5)
- added R5: 1K, Resistor_SMD:R_0805_2012Metric_Pad1.15x1.40mm_HandSolder, B.Cu at (101.0, 110.5)
- added R5: 1K, Resistor_SMD:R_0805_2012Metric_Pad1.15x1.40mm_HandSolder, B.Cu at (31.0, 110.5)
- added R5: 1K, Resistor_SMD:R_0805_2012Metric_Pad1.15x1.40mm_HandSolder, B.Cu at (171.0, 40.5)
- added R5: 1K, Resistor_SMD:R_0805_2012Metric_Pad1.15x1.40mm_HandSolder, B.Cu at (101.0, 40.5)
- added R6: 2K, Resistor_SMD:R_0805_2012Metric_Pad1.15x1.40mm_HandSolder, B.Cu at (31.0, 113.5)
- added R6: 2K, Resistor_SMD:R_0805_2012Metric_Pad1.15x1.40mm_HandSolder, B.Cu at (171.0, 113.5)
- added R6: 2K, Resistor_SMD:R_0805_2012Metric_Pad1.15x1.40mm_HandSolder, B.Cu at (101.0, 113.5)
- added R6: 2K, Resistor_SMD:R_0805_2012Metric_Pad1.15x1.40mm_HandSolder, B.Cu at (171.0, 43.5)
- added R6: 2K, Resistor_SMD:R_0805_2012Metric_Pad1.15x1.40mm_HandSolder, B.Cu at (101.0, 43.5)
- added R7: 1K, Resistor_SMD:R_0805_2012Metric_Pad1.15x1.40mm_HandSolder, B.Cu at (102.0, 120.0)
- added R7: 1K, Resistor_SMD:R_0805_2012Metric_Pad1.15x1.40mm_HandSolder, B.Cu at (32.0, 120.0)
- added R7: 1K, Resistor_SMD:R_0805_2012Metric_Pad1.15x1.40mm_HandSolder, B.Cu at (172.0, 120.0)
- added R7: 1K, Resistor_SMD:R_0805_2012Metric_Pad1.15x1.40mm_HandSolder, B.Cu at (172.0, 50.0)
- added R7: 1K, Resistor_SMD:R_0805_2012Metric_Pad1.15x1.40mm_HandSolder, B.Cu at (102.0, 50.0)
- added R8: 2K, Resistor_SMD:R_0805_2012Metric_Pad1.15x1.40mm_HandSolder, B.Cu at (102.0, 123.0)
- added R8: 2K, Resistor_SMD:R_0805_2012Metric_Pad1.15x1.40mm_HandSolder, B.Cu at (172.0, 123.0)
- added R8: 2K, Resistor_SMD:R_0805_2012Metric_Pad1.15x1.40mm_HandSolder, B.Cu at (32.0, 123.0)
- added R8: 2K, Resistor_SMD:R_0805_2012Metric_Pad1.15x1.40mm_HandSolder, B.Cu at (172.0, 53.0)
- added R8: 2K, Resistor_SMD:R_0805_2012Metric_Pad1.15x1.40mm_HandSolder, B.Cu at (102.0, 53.0)
- added R9: 1K, Resistor_SMD:R_0805_2012Metric_Pad1.15x1.40mm_HandSolder, B.Cu at (31.0, 144.0)
- added R9: 1K, Resistor_SMD:R_0805_2012Metric_Pad1.15x1.40mm_HandSolder, B.Cu at (101.0, 144.0)
- added R9: 1K, Resistor_SMD:R_0805_2012Metric_Pad1.15x1.40mm_HandSolder, B.Cu at (171.0, 144.0)
- added R9: 1K, Resistor_SMD:R_0805_2012Metric_Pad1.15x1.40mm_HandSolder, B.Cu at (171.0, 74.0)
- added R9: 1K, Resistor_SMD:R_0805_2012Metric_Pad1.15x1.40mm_HandSolder, B.Cu at (101.0, 74.0)
- added U1: DC-DC, MyFootprint:miniDCDC, F.Cu at (146.5, 113.5)
- added U1: DC-DC, MyFootprint:miniDCDC, F.Cu at (216.5, 113.5)
- added U1: DC-DC, MyFootprint:miniDCDC, F.Cu at (76.5, 113.5)
- added U1: DC-DC, MyFootprint:miniDCDC, F.Cu at (216.5, 43.5)
- added U1: DC-DC, MyFootprint:miniDCDC, F.Cu at (146.5, 43.5)
- added U2: STM32F103C8T6, MyFootprint:stm32f103c8t6-module-china, F.Cu at (44.0, 116.5)
- added U2: STM32F103C8T6, MyFootprint:stm32f103c8t6-module-china, F.Cu at (184.0, 116.5)
- added U2: STM32F103C8T6, MyFootprint:stm32f103c8t6-module-china, F.Cu at (114.0, 116.5)
- added U2: STM32F103C8T6, MyFootprint:stm32f103c8t6-module-china, F.Cu at (184.0, 46.5)
- added U2: STM32F103C8T6, MyFootprint:stm32f103c8t6-module-china, F.Cu at (114.0, 46.5)
- added U3: TB6612FNG, MyFootprint:TB6612FNG, F.Cu at (196.5, 123.5)
- added U3: TB6612FNG, MyFootprint:TB6612FNG, F.Cu at (126.5, 123.5)
- added U3: TB6612FNG, MyFootprint:TB6612FNG, F.Cu at (56.5, 123.5)
- added U3: TB6612FNG, MyFootprint:TB6612FNG, F.Cu at (196.5, 53.5)
- added U3: TB6612FNG, MyFootprint:TB6612FNG, F.Cu at (126.5, 53.5)
- moved J1 107.7 mm to (72.5, 49.5)
- moved J10 107.7 mm to (58.5, 49.5)
- moved J2 107.7 mm to (57.5, 29.5)
- moved J3 107.7 mm to (25.5, 26.6)
- moved J4 107.7 mm to (25.5, 36.1)
- moved J5 107.7 mm to (25.5, 45.6)
- moved J6 107.7 mm to (25.5, 55.1)
- moved J7 107.7 mm to (25.5, 74.0)
- moved J8 107.7 mm to (25.5, 64.5)
- moved J9 107.7 mm to (65.5, 49.5)
- moved R1 107.7 mm to (32.5, 21.5)
- moved R10 107.7 mm to (31.0, 71.5)
- moved R11 107.7 mm to (31.0, 65.0)
- moved R12 107.7 mm to (31.0, 62.0)
- moved R2 107.7 mm to (32.5, 24.5)
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Routing:
- net +5V: track 200.8 -> 1204.5 mm
- net /TXD: track 57.6 -> 345.8 mm
- net /RXD: track 45.5 -> 272.9 mm
- net /A9: track 36.3 -> 217.9 mm
- net /OUT5M: track 35.8 -> 214.6 mm
- net /VIM: track 31.8 -> 190.9 mm
- net /A10: track 31.8 -> 190.8 mm
- net /A8: track 27.2 -> 162.9 mm
- net /B14: track 25.4 -> 152.6 mm
- net /A15: track 24.7 -> 148.4 mm
- net /B13: track 22.8 -> 136.8 mm
- net /OUT6M: track 21.6 -> 129.4 mm
- net /B12: track 17.0 -> 101.7 mm
- net /OUT4M: track 15.7 -> 94.2 mm
- net /OUT1M: track 12.2 -> 73.3 mm
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Other:
- board size 56 x 57 mm -> 196 x 127 mm
